File: sms-umd/sms-umd.kicad_pcb (KiCad board)
At the start: 2 copper layers, 26.7 x 94.6 mm, 4 parts, among them CON101 UMDv3-CONN, CON102 SMS-CONN, U101 MCP23008T-E_SS

Commit message: version 3.0
Parts:
- added logo101: dblogo, db-artwork:db-logo_10mm, F.Cu at (135.9, 58.8)
Connections:
- CON101 pad 22: unconnected-(CON101A-IO0-Pad22) -> /~{M1}
- CON101 pad 23: unconnected-(CON101A-IO2-Pad23) -> /~{MC-F}
- CON101 pad 4: unconnected-(CON101A-MOSI/IO6-Pad4) -> /~{M8-B}
- CON101 pad 42: unconnected-(CON101B-IO3-Pad42) -> /~{BUSACK}
- CON101 pad 43: unconnected-(CON101B-IO1-Pad43) -> /~{BUSREQ}
- CON101 pad 5: unconnected-(CON101A-SCK/IO4-Pad5) -> /~{M0-7}
- CON102 pad 11: unconnected-(CON102-~{M0-7}-Pad11) -> /~{M0-7}
- CON102 pad 37: unconnected-(CON102-~{M1}-Pad37) -> /~{M1}
- CON102 pad 44: unconnected-(CON102-~{BUSREQ}-Pad44) -> /~{BUSREQ}
- CON102 pad 45: unconnected-(CON102-~{BUSACK}-Pad45) -> /~{BUSACK}
- CON102 pad 49: unconnected-(CON102-~{MC-F}-Pad49) -> /~{MC-F}
- CON102 pad 5: unconnected-(CON102-~{M8-B}-Pad5) -> /~{M8-B}
Routing:
- net /~{RST}: track 0.00 -> 115.4 mm, vias 0 -> 1
- net /CLK: track 0.00 -> 73.9 mm, vias 0 -> 2
- net /~{MREQ}: track 0.00 -> 57.6 mm, vias 0 -> 1
- net /A12: track 0.00 -> 49.5 mm, vias 0 -> 2
- net /~{CE}: track 0.00 -> 49.4 mm
- net /A15: track 0.00 -> 47.2 mm, vias 0 -> 2
- net /A0: track 0.00 -> 42.2 mm
- net /A2: track 0.00 -> 41.1 mm, vias 0 -> 1
- net /A4: track 0.00 -> 39.3 mm, vias 0 -> 1
- net /A1: track 0.00 -> 37.8 mm, vias 0 -> 3
- net /~{WR}: track 0.00 -> 34.5 mm
- net /A3: track 0.00 -> 33.3 mm, vias 0 -> 3
- net /5V_1: track 0.00 -> 30.8 mm
- net /D4: track 0.00 -> 30.1 mm
- net /D5: track 0.00 -> 28.9 mm, vias 0 -> 2
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