File: sms-umd/sms-umd.kicad_sch (KiCad schematic)
At the start: 4 parts, among them CON101 UMDv3-CONN, CON102 SMS-CONN, U101 MCP23008T-E_SS

Commit message: version 3.0
Parts:
- added logo101: dblogo, db-artwork:db-logo_10mm, symbol db-artwork:logo
Connections:
- net ~{M0-7}: now reaches CON102.11 (~{M0-7})
- net ~{M0-7}: now also CON101.5 (SCK/IO4)
- net ~{M1}: now reaches CON102.37 (~{M1})
- net ~{M1}: now also CON101.22 (IO0)
- net ~{BUSREQ}: now reaches CON102.44 (~{BUSREQ})
- net ~{BUSREQ}: now also CON101.43 (IO1)
- net ~{BUSACK}: now reaches CON102.45 (~{BUSACK})
- net ~{BUSACK}: now also CON101.42 (IO3)
- net ~{MC-F}: now reaches CON102.49 (~{MC-F})
- net ~{MC-F}: now also CON101.23 (IO2)
- net ~{M8-B}: now reaches CON102.5 (~{M8-B})
- net ~{M8-B}: now also CON101.4 (MOSI/IO6)
Changed lines of the file:
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@@
   (title_block
     (title "Sega Master System UMDv3 Cartridge Adapter")
-    (date "2023-11-17")
+    (date "2023-12-20")
     (rev "3.0")
     (company "db Electronics")
@@
     (stroke (width 0) (type default))
   )
+  (wire (pts (xy 114.3 54.61) (xy 128.27 54.61))
+    (stroke (width 0) (type default))
+  )
   (wire (pts (xy 113.03 157.48) (xy 116.84 157.48))
     (stroke (width 0) (type default))
@@
     (stroke (width 0) (type default))
   )
+  (wire (pts (xy 73.66 59.69) (xy 87.63 59.69))
+    (stroke (width 0) (type default))
+  )
   (wire (pts (xy 114.3 72.39) (xy 125.73 72.39))
     (stroke (width 0) (type default))
@@
     (stroke (width 0) (type default))
   )
+  (wire (pts (xy 114.3 105.41) (xy 128.27 105.41))
+    (stroke (width 0) (type default))
+  )
   (wire (pts (xy 113.03 172.72) (xy 119.38 172.72))
     (stroke (width 0) (type default))
@@
     (stroke (width 0) (type default))
   )
+  (wire (pts (xy 195.58 102.87) (xy 209.55 102.87))
+    (stroke (width 0) (type default))
+  )
   (wire (pts (xy 73.66 77.47) (xy 87.63 77.47))
     (stroke (width 0) (type default))
@@
     (stroke (width 0) (type default))
   )
+  (wire (pts (xy 73.66 105.41) (xy 87.63 105.41))
+    (stroke (width 0) (type default))
+  )
   (wire (pts (xy 73.66 118.11) (xy 87.63 118.11))
     (stroke (width 0) (type default))
@@
     (stroke (width 0) (type default))
   )
+  (wire (pts (xy 153.67 102.87) (xy 167.64 102.87))
+    (stroke (width 0) (type default))
+  )
   (wire (pts (xy 195.58 118.11) (xy 209.55 118.11))
     (stroke (width 0) (type default))
@@
     (stroke (width 0) (type default))
   )
+  (wire (pts (xy 73.66 57.15) (xy 87.63 57.15))
+    (stroke (width 0) (type default))
+  )
   (wire (pts (xy 153.67 52.07) (xy 167.64 52.07))
     (stroke (width 0) (type default))
@@
     (stroke (width 0) (type default))
   )
+  (wire (pts (xy 114.3 95.25) (xy 128.27 95.25))
+    (stroke (width 0) (type default))
+  )
   (wire (pts (xy 128.27 74.93) (xy 125.73 74.93))
     (stroke (width 0) (type default))
@@
     (stroke (width 0) (type default))
   )
+  (wire (pts (xy 114.3 110.49) (xy 128.27 110.49))
+    (stroke (width 0) (type default))
+  )
   (wire (pts (xy 82.55 167.64) (xy 82.55 170.18))
     (stroke (width 0) (type default))
@@
     (stroke (width 0) (type default))
   )
+  (wire (pts (xy 195.58 105.41) (xy 209.55 105.41))
+    (stroke (width 0) (type default))
+  )
   (wire (pts (xy 195.58 54.61) (xy 209.55 54.61))
     (stroke (width 0) (type default))
@@
     (stroke (width 0) (type default))
   )
+  (wire (pts (xy 114.3 62.23) (xy 128.27 62.23))
+    (stroke (width 0) (type default))
+  )
   (wire (pts (xy 34.29 184.15) (xy 34.29 182.88))
     (stroke (width 0) (type default))
@@
   )
   (wire (pts (xy 86.36 167.64) (xy 82.55 167.64))
+    (stroke (width 0) (type default))
+  )
+  (wire (pts (xy 73.66 102.87) (xy 87.63 102.87))
     (stroke (width 0) (type default))
   )
@@
     (effects (font (size 1.27 1.27)) (justify left bottom))
   )
+  (label "~{MC-F}" (at 114.3 110.49 0) (fields_autoplaced)
+    (effects (font (size 1.27 1.27)) (justify left bottom))
+  )
+  (label "~{M1}" (at 114.3 95.25 0) (fields_autoplaced)
+    (effects (font (size 1.27 1.27)) (justify left bottom))
+  )
   (label "5V_1" (at 195.58 125.73 0) (fields_autoplaced)
     (effects (font (size 1.27 1.27)) (justify left bottom))
@@
     (effects (font (size 1.27 1.27)) (justify left bottom))
   )
+  (label "~{M0-7}" (at 74.93 59.69 0) (fields_autoplaced)
+    (effects (font (size 1.27 1.27)) (justify left bottom))
+  )
   (label "GND" (at 195.58 49.53 0) (fields_autoplaced)
     (effects (font (size 1.27 1.27)) (justify left bottom))
@@
     (effects (font (size 1.27 1.27)) (justify left bottom))
   )
+  (label "~{BUSACK}" (at 114.3 105.41 0) (fields_autoplaced)
+    (effects (font (size 1.27 1.27)) (justify left bottom))
+  )
   (label "D6" (at 114.3 67.31 0) (fields_autoplaced)
     (effects (font (size 1.27 1.27)) (justify left bottom))
@@
     (effects (font (size 1.27 1.27)) (justify left bottom))
   )
+  (label "~{MC-F}" (at 74.93 105.41 0) (fields_autoplaced)
+    (effects (font (size 1.27 1.27)) (justify left bottom))
+  )
   (label "CLK" (at 195.58 62.23 0) (fields_autoplaced)
     (effects (font (size 1.27 1.27)) (justify left bottom))
@@
     (effects (font (size 1.27 1.27)) (justify left bottom))
   )
+  (label "~{BUSREQ}" (at 154.94 102.87 0) (fields_autoplaced)
+    (effects (font (size 1.27 1.27)) (justify left bottom))
+  )
+  (label "~{M0-7}" (at 114.3 62.23 0) (fields_autoplaced)
+    (effects (font (size 1.27 1.27)) (justify left bottom))
+  )
+  (label "~{M1}" (at 74.93 102.87 0) (fields_autoplaced)
+    (effects (font (size 1.27 1.27)) (justify left bottom))
+  )
   (label "A1" (at 74.93 118.11 0) (fields_autoplaced)
     (effects (font (size 1.27 1.27)) (justify left bottom))
@@
     (effects (font (size 1.27 1.27)) (justify left bottom))
   )
+  (label "~{BUSACK}" (at 195.58 105.41 0) (fields_autoplaced)
+    (effects (font (size 1.27 1.27)) (justify left bottom))
+  )
   (label "5V_0" (at 114.3 49.53 0) (fields_autoplaced)
     (effects (font (size 1.27 1.27)) (justify left bottom))
@@
     (effects (font (size 1.27 1.27)) (justify left bottom))
   )
+  (label "~{M8-B}" (at 114.3 54.61 0) (fields_autoplaced)
+    (effects (font (size 1.27 1.27)) (justify left bottom))
+  )
   (label "~{IORQ}" (at 195.58 110.49 0) (fields_autoplaced)
     (effects (font (size 1.27 1.27)) (justify left bottom))
@@
     (effects (font (size 1.27 1.27)) (justify left bottom))
   )
+  (label "~{M8-B}" (at 74.93 57.15 0) (fields_autoplaced)
+    (effects (font (size 1.27 1.27)) (justify left bottom))
+  )
   (label "A13" (at 74.93 67.31 0) (fields_autoplaced)
     (effects (font (size 1.27 1.27)) (justify left bottom))
@@
   )
   (label "A10" (at 74.93 77.47 0) (fields_autoplaced)
+    (effects (font (size 1.27 1.27)) (justify left bottom))
+  )
+  (label "~{BUSREQ}" (at 195.58 102.87 0) (fields_autoplaced)
     (effects (font (size 1.27 1.27)) (justify left bottom))
   )
@@
         )
       )
+    )
+  )
+  (symbol (lib_id "db-artwork:logo") (at 167.005 151.765 0) (unit 1)
+    (in_bom yes) (on_board yes) (dnp no) (fields_autoplaced)
+    (property "Reference" "logo101" (at 172.72 150.495 0)
+      (effects (font (size 1.524 1.524)) (justify left))
+    )
+    (property "Value" "dblogo" (at 172.72 153.035 0)
+      (effects (font (size 1.524 1.524)) (justify left))
+    )
+    (property "Footprint" "db-artwork:db-logo_10mm" (at 167.005 151.765 0)
+      (effects (font (size 1.524 1.524)) hide)
+    )
+    (property "Datasheet" "" (at 167.005 151.765 0)
+      (effects (font (size 1.524 1.524)) hide)
+    )
+    (instances
+      (project "sms-umd"
+        (path "/89a61d91-e45c-44db-8631-8ab2706d2cb9"
+          (reference "logo101") (unit 1)
+        )
+      )
